Commit message: Added ros2 control for gazebo

File: autoserve_description/urdf/autoserve.xacro (robot description, xacro)
@@ -3,13 +3,13 @@
 <xacro:include filename="$(find autoserve_description)/urdf/materials.xacro" />
 <xacro:include filename="$(find autoserve_description)/urdf/autoserve_gazebo.xacro" />
-<xacro:include filename="$(find autoserve_description)/urdf/autoserve_ros2_control.xacro" />
+<!-- <xacro:include filename="$(find autoserve_description)/urdf/autoserve_ros2_control.xacro" /> -->
 <xacro:include filename="$(find autoserve_description)/urdf/autoserve.trans" />
 <link name="base_footprint">
-  <collision>
-    <origin xyz="0.0 0.0 0.006" rpy="0 0 0"/>
-    <geometry>
-      <box size="0.40 0.20 0.01" />
-    </geometry>
-  </collision>
+  <!-- <collision>
+    <origin xyz="0.0 0.0 0.05" rpy="0 0 0"/>
+    <geometry>
+      <box size="0.45 0.20 0.01" />
+    </geometry>
+  </collision> -->
 </link>
 <link name="base_link">
@@ -26,8 +26,14 @@
     <material name="plastic_translucent_matte_green"/>
   </visual>
-  <collision>
+  <!-- <collision>
     <origin xyz="0 0 0" rpy="0 0 0"/>
     <geometry>
       <mesh filename="package://autoserve_description/meshes/base_link.stl" scale="0.001 0.001 0.001"/>
+    </geometry>
+  </collision> -->
+  <collision>
+    <origin xyz="0.0 0.0 0.008" rpy="0 0 0"/>
+    <geometry>
+      <box size="0.40 0.20 0.01" />
     </geometry>
   </collision>
@@ -99,5 +105,5 @@
   </collision>
 </link>
-<link name="depth_camera_2">
+<!-- <link name="depth_camera_2">
   <inertial>
     <origin xyz="0.01195115490287238 0.02274721773464422 -6.09413650859425e-05" rpy="0 0 0"/>
@@ -118,4 +124,24 @@
     </geometry>
   </collision>
+</link> -->
+<link name="depth_camera_2">
+  <inertial>
+    <origin xyz="0.01195115490287238 0.02274721773464422 -6.09413650859425e-05" rpy="0 0 0"/>
+    <mass value="0.35132131581082054"/>
+    <inertia ixx="0.000227" iyy="3.2e-05" izz="0.000229" ixy="-1e-06" iyz="-0.0" ixz="-0.0"/>
+  </inertial>
+  <visual>
+    <origin xyz="-0.105108 0.0 -0.771167" rpy="0 0 0"/>
+    <geometry>
+      <mesh filename="package://autoserve_description/meshes/depth_camera_v1_2.stl" scale="0.001 0.001 0.001"/>
+    </geometry>
+    <material name="plastic_translucent_matte_red"/>
+  </visual>
+  <collision>
+    <origin xyz="-0.105108 0.0 -0.771167" rpy="0 0 0"/>
+    <geometry>
+      <mesh filename="package://autoserve_description/meshes/depth_camera_v1_2.stl" scale="0.001 0.001 0.001"/>
+    </geometry>
+  </collision>
 </link>
 <link name="right_wheel">
@@ -214,11 +240,16 @@
   <child link="depth_camera_1"/>
 </joint>
+<!-- <joint name="base2camera_2" type="fixed">
+  <origin xyz="0.105108 -0.0 0.771167" rpy="0 0 0"/>
+  <parent link="base_link"/>
+  <child link="depth_camera_2"/>
+</joint> -->
 <joint name="base2camera_2" type="fixed">
-  <origin xyz="0.105108 -0.0 0.771167" rpy="0 0 0"/>
+  <origin xyz="0.105108 -0.0 1.3" rpy="0 0 0"/>
   <parent link="base_link"/>
   <child link="depth_camera_2"/>
 </joint>
 <joint name="base2rightw" type="continuous">
-  <origin xyz="0.0 -0.1659 0.05" rpy="0 0 0"/>
+  <origin xyz="0.0 -0.17 0.05" rpy="0 0 0"/>
   <parent link="base_link"/>
   <child link="right_wheel"/>
@@ -226,5 +257,5 @@
 </joint>
 <joint name="base2leftw" type="continuous">
-  <origin xyz="0.0 0.1659 0.05" rpy="0 0 0"/>
+  <origin xyz="0.0 0.17 0.05" rpy="0 0 0"/>
   <parent link="base_link"/>
   <child link="left_wheel"/>

File: autoserve_description/urdf/autoserve_gazebo.xacro (robot description, xacro)
@@ -31,19 +31,13 @@
   <gazebo reference="base_link">
     <material>${base_link}</material>
-    <mu1>0.1</mu1>
-    <mu2>0.1</mu2>
-    <kp>1000000.0</kp>
-    <kd>100.0</kd>
-    <minDepth>0.001</minDepth>
-    <maxVel>1.0</maxVel>
+    <mu1>0.01</mu1>
+    <mu2>0.01</mu2>
+    <gravity>true</gravity>
   </gazebo>
   <gazebo reference="base_footprint">
     <material>${base_link}</material>
-    <mu1>0.1</mu1>
-    <mu2>0.1</mu2>
-    <kp>1000000.0</kp>
-    <kd>100.0</kd>
-    <minDepth>0.001</minDepth>
-    <maxVel>1.0</maxVel>
+    <mu1>0.01</mu1>
+    <mu2>0.01</mu2>
+    <gravity>true</gravity>
   </gazebo>
   <gazebo reference="depth_camera_1">
@@ -51,8 +45,5 @@
     <mu1>0.1</mu1>
     <mu2>0.1</mu2>
-    <kp>1000000.0</kp>
-    <kd>100.0</kd>
-    <minDepth>0.001</minDepth>
-    <maxVel>1.0</maxVel>
+    <gravity>true</gravity>
   </gazebo>
   <gazebo reference="depth_camera_2">
@@ -60,8 +51,5 @@
     <mu1>0.1</mu1>
     <mu2>0.1</mu2>
-    <kp>1000000.0</kp>
-    <kd>100.0</kd>
-    <minDepth>0.001</minDepth>
-    <maxVel>1.0</maxVel>
+    <gravity>true</gravity>
   </gazebo>
   <gazebo reference="ydlidar">
@@ -69,31 +57,28 @@
     <mu1>0.1</mu1>
     <mu2>0.1</mu2>
-    <kp>1000000.0</kp>
-    <kd>100.0</kd>
-    <minDepth>0.001</minDepth>
-    <maxVel>1.0</maxVel>
+    <gravity>true</gravity>
+  </gazebo>
+  <gazebo reference="imu">
+    <material>${imu}</material>
+    <mu1>0.1</mu1>
+    <mu2>0.1</mu2>
+    <gravity>true</gravity>
   </gazebo>
   <gazebo reference="plate_1">
     <material>${plate}</material>
-    <mu1>10</mu1>
-    <mu2>10</mu2>
-    <kp>1000000.0</kp>
-    <kd>100.0</kd>
-    <minDepth>0.001</minDepth>
-    <maxVel>1.0</maxVel>
+    <mu1>10.0</mu1>
+    <mu2>10.0</mu2>
+    <gravity>true</gravity>
   </gazebo>
   <gazebo reference="plate_2">
     <material>${plate}</material>
-    <mu1>10</mu1>
-    <mu2>10</mu2>
-    <kp>1000000.0</kp>
-    <kd>100.0</kd>
-    <minDepth>0.001</minDepth>
-    <maxVel>1.0</maxVel>
+    <mu1>10.0</mu1>
+    <mu2>10.0</mu2>
+    <gravity>true</gravity>
   </gazebo>
   <gazebo>
     <plugin filename="libgazebo_ros2_control.so" name="gazebo_ros2_control">
-      <robot_param>robot_description</robot_param>
-      <robot_param_node>robot_state_publisher</robot_param_node>
+      <!-- <robot_param>robot_description</robot_param>
+      <robot_param_node>robot_state_publisher</robot_param_node> -->
       <parameters>$(find autoserve_controller)/config/autoserve_controllers.yaml</parameters>
     </plugin>
@@ -113,9 +98,9 @@
       <!-- output -->
       <publish_odom>true</publish_odom>
-      <publish_odom_tf>true</publish_odom_tf>
-      <publish_wheel_tf>true</publish_wheel_tf>
+      <publish_odom_tf>false</publish_odom_tf>
+      <publish_wheel_tf>false</publish_wheel_tf>
       <odometry_topic>odom</odometry_topic>
       <odometry_frame>odom</odometry_frame>
-      <robot_base_frame>base_footprint</robot_base_frame>
+      <robot_base_frame>base_link</robot_base_frame>
     </plugin>
   </gazebo>

File: autoserve_description/urdf/autoserve_ros2_control.xacro (robot description, xacro)
@@ -1,4 +1,4 @@
 <?xml version="1.0"?>
-<robot xmlns:xacro="http://www.ros.org/wiki/xacro" name="autoserve">
+<robot xmlns:xacro="http://www.ros.org/wiki/xacro" name="autoserve_ros2">
     <ros2_control name="RobotSystem" type="system">
         <hardware>
@@ -19,4 +19,20 @@
             <state_interface name="position" />
         </joint>
+        <joint name="base2leftw">
+            <command_interface name="velocity">
+              <param name="min">-1</param>
+              <param name="max">1</param>
+            </command_interface>
+            <state_interface name="position" />
+            <state_interface name="velocity" />
+        </joint>
+        <joint name="base2rightw">
+            <command_interface name="velocity">
+              <param name="min">-1</param>
+              <param name="max">1</param>
+            </command_interface>
+            <state_interface name="position" />
+            <state_interface name="velocity" />
+        </joint>
     </ros2_control>
 </robot>

Commit message: Updated simulation

File: autoserve_description/urdf/autoserve.xacro (robot description, xacro)
@@ -6,10 +6,10 @@
 <xacro:include filename="$(find autoserve_description)/urdf/autoserve.trans" />
 <link name="base_footprint">
-  <!-- <collision>
-    <origin xyz="0.0 0.0 0.05" rpy="0 0 0"/>
+  <collision>
+    <origin xyz="0.0 0.0 0.006" rpy="0 0 0"/>
     <geometry>
       <box size="0.45 0.20 0.01" />
     </geometry>
-  </collision> -->
+  </collision>
 </link>
 <link name="base_link">
@@ -26,16 +26,16 @@
     <material name="plastic_translucent_matte_green"/>
   </visual>
+  <collision>
+    <origin xyz="0 0 0" rpy="0 0 0"/>
+    <geometry>
+      <mesh filename="package://autoserve_description/meshes/base_link.stl" scale="0.001 0.001 0.001"/>
+    </geometry>
+  </collision>
   <!-- <collision>
-    <origin xyz="0 0 0" rpy="0 0 0"/>
-    <geometry>
-      <mesh filename="package://autoserve_description/meshes/base_link.stl" scale="0.001 0.001 0.001"/>
+    <origin xyz="0.0 0.0 0.007" rpy="0 0 0"/>
+    <geometry>
+      <box size="0.40 0.20 0.01" />
     </geometry>
   </collision> -->
-  <collision>
-    <origin xyz="0.0 0.0 0.008" rpy="0 0 0"/>
-    <geometry>
-      <box size="0.40 0.20 0.01" />
-    </geometry>
-  </collision>
 </link>
 <joint name="footprint2baselink" type="fixed">
@@ -148,5 +148,5 @@
   <inertial>
     <origin xyz="1.4446033464149508e-16 -0.015000000000000263 2.0816681711721685e-16" rpy="0 0 0"/>
-    <mass value="0.028210189769456086"/>
+    <mass value="1.528210189769456086"/>
     <inertia ixx="2e-05" iyy="3.5e-05" izz="2e-05" ixy="-0.0" iyz="0.0" ixz="0.0"/>
   </inertial>
@@ -168,5 +168,5 @@
   <inertial>
     <origin xyz="1.6623077439054263e-16 0.01500000000000018 1.3877787807814457e-16" rpy="0 0 0"/>
-    <mass value="0.028210189769456086"/>
+    <mass value="1.528210189769456086"/>
     <inertia ixx="2e-05" iyy="3.5e-05" izz="2e-05" ixy="0.0" iyz="0.0" ixz="0.0"/>
   </inertial>
@@ -251,11 +251,11 @@
 </joint>
 <joint name="base2rightw" type="continuous">
-  <origin xyz="0.0 -0.17 0.05" rpy="0 0 0"/>
+  <origin xyz="0.0 -0.1659 0.05" rpy="0 0 0"/>
   <parent link="base_link"/>
   <child link="right_wheel"/>
-  <axis xyz="-0.0 1.0 -0.0"/>
+  <axis xyz="-0.0 1.0 0.0"/>
 </joint>
 <joint name="base2leftw" type="continuous">
-  <origin xyz="0.0 0.17 0.05" rpy="0 0 0"/>
+  <origin xyz="0.0 0.1659 0.05" rpy="0 0 0"/>
   <parent link="base_link"/>
   <child link="left_wheel"/>

File: autoserve_description/urdf/autoserve_gazebo.xacro (robot description, xacro)
@@ -1,5 +1,5 @@
 <?xml version="1.0"?>
 <robot name="autonav" xmlns:xacro="http://ros.org/wiki/xacro">
-<xacro:property name="base_link" value="Gazebo/FlatBlack" />
+<xacro:property name="base_link" value="Gazebo/Red" />
 <xacro:property name="wheels" value="Gazebo/Black" />
 <xacro:property name="imu" value="Gazebo/PurpleGlow" />
@@ -10,34 +10,31 @@
   <gazebo reference="left_wheel">
     <material>${wheels}</material>
-    <mu1>1000000000000000.0</mu1>
-    <mu2>1000000000000000.0</mu2>
-    <kp>1000000000000.0</kp>
-    <kd>10.0</kd>
-    <minDepth>0.001</minDepth>
-    <maxVel>0.1</maxVel>
-    <fdir1>1 0 0</fdir1>
+    <mu1>1000.0</mu1>
+    <mu2>1000.0</mu2>
+    <maxContacts>1</maxContacts>
+    <selfCollide>true</selfCollide>
+    <gravity>true</gravity>
   </gazebo>
   <gazebo reference="right_wheel">
     <material>${wheels}</material>
-    <mu1>1000000000000000.0</mu1>
-    <mu2>1000000000000000.0</mu2>
-    <kp>1000000000000.0</kp>
-    <kd>10.0</kd>
-    <minDepth>0.001</minDepth>
-    <maxVel>0.1</maxVel>
-    <fdir1>1 0 0</fdir1>
+    <mu1>1000.0</mu1>
+    <mu2>1000.0</mu2>
+    <maxContacts>1</maxContacts>
+    <selfCollide>true</selfCollide>
+    <gravity>true</gravity>
   </gazebo>
   <!-- Caster Wheels -->
   <gazebo reference="base_link">
     <material>${base_link}</material>
-    <mu1>0.01</mu1>
-    <mu2>0.01</mu2>
+    <mu1>0.1</mu1>
+    <mu2>0.1</mu2>
+    <maxContacts>1</maxContacts>
+    <selfCollide>true</selfCollide>
     <gravity>true</gravity>
   </gazebo>
   <gazebo reference="base_footprint">
-    <material>${base_link}</material>
-    <mu1>0.01</mu1>
-    <mu2>0.01</mu2>
-    <gravity>true</gravity>
+    <mu1>0.1</mu1>
+    <mu2>0.1</mu2>
+    <maxContacts>1</maxContacts>
   </gazebo>
   <gazebo reference="depth_camera_1">
@@ -45,5 +42,4 @@
     <mu1>0.1</mu1>
     <mu2>0.1</mu2>
-    <gravity>true</gravity>
   </gazebo>
   <gazebo reference="depth_camera_2">
@@ -51,5 +47,4 @@
     <mu1>0.1</mu1>
     <mu2>0.1</mu2>
-    <gravity>true</gravity>
   </gazebo>
   <gazebo reference="ydlidar">
@@ -57,5 +52,4 @@
     <mu1>0.1</mu1>
     <mu2>0.1</mu2>
-    <gravity>true</gravity>
   </gazebo>
   <gazebo reference="imu">
@@ -63,22 +57,19 @@
     <mu1>0.1</mu1>
     <mu2>0.1</mu2>
-    <gravity>true</gravity>
   </gazebo>
   <gazebo reference="plate_1">
     <material>${plate}</material>
-    <mu1>10.0</mu1>
-    <mu2>10.0</mu2>
-    <gravity>true</gravity>
+    <mu1>0.1</mu1>
+    <mu2>0.1</mu2>
   </gazebo>
   <gazebo reference="plate_2">
     <material>${plate}</material>
-    <mu1>10.0</mu1>
-    <mu2>10.0</mu2>
-    <gravity>true</gravity>
+    <mu1>0.1</mu1>
+    <mu2>0.1</mu2>
   </gazebo>
   <gazebo>
     <plugin filename="libgazebo_ros2_control.so" name="gazebo_ros2_control">
-      <!-- <robot_param>robot_description</robot_param>
-      <robot_param_node>robot_state_publisher</robot_param_node> -->
+      <robot_param>robot_description</robot_param>
+      <robot_param_node>robot_state_publisher</robot_param_node>
       <parameters>$(find autoserve_controller)/config/autoserve_controllers.yaml</parameters>
     </plugin>
@@ -86,21 +77,16 @@
   <gazebo>
     <plugin name="diff_drive_control" filename="libgazebo_ros_diff_drive.so">
-      <!-- Update rate in Hz -->
       <update_rate>50</update_rate>
-      <!-- wheels -->
       <left_joint>base2leftw</left_joint>
       <right_joint>base2rightw</right_joint>
-      <!-- kinematics -->
       <wheel_separation>0.34</wheel_separation>
       <wheel_diameter>0.1</wheel_diameter>
-      <!-- input -->
       <command_topic>cmd_vel</command_topic>
-      <!-- output -->
       <publish_odom>true</publish_odom>
-      <publish_odom_tf>false</publish_odom_tf>
-      <publish_wheel_tf>false</publish_wheel_tf>
+      <publish_odom_tf>true</publish_odom_tf>
+      <publish_wheel_tf>true</publish_wheel_tf>
       <odometry_topic>odom</odometry_topic>
       <odometry_frame>odom</odometry_frame>
-      <robot_base_frame>base_link</robot_base_frame>
+      <robot_base_frame>base_footprint</robot_base_frame>
     </plugin>
   </gazebo>
@@ -134,5 +120,5 @@
         </scan>
         <range>
-          <min>0.10</min>
+          <min>0.5</min>
           <max>30.0</max>
           <resolution>0.01</resolution>
@@ -158,5 +144,5 @@
         <min_intensity>100.0</min_intensity>
         <!-- Frame id for header of output, defaults to sensor's parent link name -->
-        <frame_name>lidar</frame_name>
+        <frame_name>ydlidar</frame_name>
       </plugin>
     </sensor>

File: autoserve_description/urdf/autoserve_ros2_control.xacro (robot description, xacro)
@@ -1,5 +1,5 @@
 <?xml version="1.0"?>
-<robot xmlns:xacro="http://www.ros.org/wiki/xacro" name="autoserve_ros2">
-    <ros2_control name="RobotSystem" type="system">
+<robot xmlns:xacro="http://www.ros.org/wiki/xacro" name="autoserve">
+    <ros2_control name="autoserve" type="system">
         <hardware>
             <plugin>gazebo_ros2_control/GazeboSystem</plugin>
@@ -19,8 +19,8 @@
             <state_interface name="position" />
         </joint>
-        <joint name="base2leftw">
+        <!-- <joint name="base2leftw">
             <command_interface name="velocity">
-              <param name="min">-1</param>
-              <param name="max">1</param>
+              <param name="min">-10</param>
+              <param name="max">10</param>
             </command_interface>
             <state_interface name="position" />
@@ -29,10 +29,10 @@
         <joint name="base2rightw">
             <command_interface name="velocity">
-              <param name="min">-1</param>
-              <param name="max">1</param>
+              <param name="min">-10</param>
+              <param name="max">10</param>
             </command_interface>
             <state_interface name="position" />
             <state_interface name="velocity" />
-        </joint>
+        </joint> -->
     </ros2_control>
 </robot>

Commit message: Added gazebo package and custom world

File: autoserve_description/urdf/autoserve.xacro (robot description, xacro)
@@ -3,13 +3,13 @@
 <xacro:include filename="$(find autoserve_description)/urdf/materials.xacro" />
 <xacro:include filename="$(find autoserve_description)/urdf/autoserve_gazebo.xacro" />
-<!-- <xacro:include filename="$(find autoserve_description)/urdf/autoserve_ros2_control.xacro" /> -->
+<xacro:include filename="$(find autoserve_description)/urdf/autoserve_ros2_control.xacro" />
 <xacro:include filename="$(find autoserve_description)/urdf/autoserve.trans" />
 <link name="base_footprint">
-  <collision>
-    <origin xyz="0.0 0.0 0.006" rpy="0 0 0"/>
+  <!-- <collision>
+    <origin xyz="0.0 0.0 0.0055" rpy="0 0 0"/>
     <geometry>
       <box size="0.45 0.20 0.01" />
     </geometry>
-  </collision>
+  </collision> -->
 </link>
 <link name="base_link">
@@ -26,16 +26,16 @@
     <material name="plastic_translucent_matte_green"/>
   </visual>
-  <collision>
+  <!-- <collision>
     <origin xyz="0 0 0" rpy="0 0 0"/>
     <geometry>
       <mesh filename="package://autoserve_description/meshes/base_link.stl" scale="0.001 0.001 0.001"/>
     </geometry>
-  </collision>
-  <!-- <collision>
-    <origin xyz="0.0 0.0 0.007" rpy="0 0 0"/>
-    <geometry>
-      <box size="0.40 0.20 0.01" />
-    </geometry>
   </collision> -->
+  <collision>
+    <origin xyz="0.0 0.0 0.006" rpy="0 0 0"/>
+    <geometry>
+      <box size="0.45 0.20 0.01" />
+    </geometry>
+  </collision>
 </link>
 <joint name="footprint2baselink" type="fixed">
@@ -105,5 +105,5 @@
   </collision>
 </link>
-<!-- <link name="depth_camera_2">
+<link name="depth_camera_2">
   <inertial>
     <origin xyz="0.01195115490287238 0.02274721773464422 -6.09413650859425e-05" rpy="0 0 0"/>
@@ -124,6 +124,6 @@
     </geometry>
   </collision>
-</link> -->
-<link name="depth_camera_2">
+</link>
+<!-- <link name="depth_camera_2">
   <inertial>
     <origin xyz="0.01195115490287238 0.02274721773464422 -6.09413650859425e-05" rpy="0 0 0"/>
@@ -144,5 +144,5 @@
     </geometry>
   </collision>
-</link>
+</link> -->
 <link name="right_wheel">
   <inertial>
@@ -240,14 +240,14 @@
   <child link="depth_camera_1"/>
 </joint>
+<joint name="base2camera_2" type="fixed">
+  <origin xyz="0.105108 -0.0 0.771167" rpy="0 0 0"/>
+  <parent link="base_link"/>
+  <child link="depth_camera_2"/>
+</joint>
 <!-- <joint name="base2camera_2" type="fixed">
-  <origin xyz="0.105108 -0.0 0.771167" rpy="0 0 0"/>
+  <origin xyz="0.105108 -0.0 1.3" rpy="0 0 0"/>
   <parent link="base_link"/>
   <child link="depth_camera_2"/>
 </joint> -->
-<joint name="base2camera_2" type="fixed">
-  <origin xyz="0.105108 -0.0 1.3" rpy="0 0 0"/>
-  <parent link="base_link"/>
-  <child link="depth_camera_2"/>
-</joint>
 <joint name="base2rightw" type="continuous">
   <origin xyz="0.0 -0.1659 0.05" rpy="0 0 0"/>
@@ -262,17 +262,18 @@
   <axis xyz="0.0 1.0 0.0"/>
 </joint>
-<joint name="base2plate_1" type="prismatic">
+<!-- prismatic -->
+<joint name="base2plate_1" type="fixed">
   <origin xyz="0.0 -0.0 0.303" rpy="0 0 0"/>
   <parent link="base_link"/>
   <child link="plate_1"/>
-  <axis xyz="1.0 -0.0 -0.0"/>
-  <limit upper="0.08" lower="-0.08" effort="100" velocity="100"/>
-</joint>
-<joint name="base2plate_2" type="prismatic">
+  <!-- <axis xyz="1.0 -0.0 -0.0"/>
+  <limit upper="0.08" lower="-0.08" effort="100" velocity="100"/> -->
+</joint>
+<joint name="base2plate_2" type="fixed">
   <origin xyz="0.0 -0.0 0.533" rpy="0 0 0"/>
   <parent link="base_link"/>
   <child link="plate_2"/>
-  <axis xyz="1.0 -0.0 -0.0"/>
-  <limit upper="0.08" lower="-0.08" effort="100" velocity="100"/>
+  <!-- <axis xyz="1.0 -0.0 -0.0"/>
+  <limit upper="0.08" lower="-0.08" effort="100" velocity="100"/> -->
 </joint>
 </robot>

File: autoserve_description/urdf/autoserve_gazebo.xacro (robot description, xacro)
@@ -1,4 +1,4 @@
 <?xml version="1.0"?>
-<robot name="autonav" xmlns:xacro="http://ros.org/wiki/xacro">
+<robot name="autoserve" xmlns:xacro="http://ros.org/wiki/xacro">
 <xacro:property name="base_link" value="Gazebo/Red" />
 <xacro:property name="wheels" value="Gazebo/Black" />
@@ -68,5 +68,5 @@
     <mu2>0.1</mu2>
   </gazebo>
-  <gazebo>
+  <!-- <gazebo>
     <plugin filename="libgazebo_ros2_control.so" name="gazebo_ros2_control">
       <robot_param>robot_description</robot_param>
@@ -74,5 +74,5 @@
       <parameters>$(find autoserve_controller)/config/autoserve_controllers.yaml</parameters>
     </plugin>
-  </gazebo>
+  </gazebo> -->
   <gazebo>
     <plugin name="diff_drive_control" filename="libgazebo_ros_diff_drive.so">
@@ -126,8 +126,4 @@
         <noise>
           <type>gaussian</type>
-          <!-- Noise parameters based on published spec for Hokuyo laser
-               achieving "+-30mm" accuracy at range < 10m.  A mean of 0.0m and
-               stddev of 0.01m will put 99.7% of samples within 0.03m of the true
-               reading. -->
           <mean>0.0</mean>
           <stddev>0.01</stddev>
@@ -136,12 +132,8 @@
       <plugin name="my_ray_sensor_plugin" filename="libgazebo_ros_ray_sensor.so">
         <ros>
-          <!-- Configure namespace and remap to publish to /ray/pointcloud2 -->
           <remapping>~/out:=scan</remapping>
         </ros>
-        <!-- Output as a PointCloud2, see above for other types -->
         <output_type>sensor_msgs/LaserScan</output_type>
-        <!-- Clip intensity values so all are above 100, optional -->
         <min_intensity>100.0</min_intensity>
-        <!-- Frame id for header of output, defaults to sensor's parent link name -->
         <frame_name>ydlidar</frame_name>
       </plugin>
