Commit message: updated urdf and gazebo world launch file

File: autoserve_description/urdf/autoserve.xacro (robot description, xacro)
@@ -3,11 +3,10 @@
 <xacro:include filename="$(find autoserve_description)/urdf/materials.xacro" />
 <xacro:include filename="$(find autoserve_description)/urdf/autoserve_gazebo.xacro" />
-<xacro:include filename="$(find autoserve_description)/urdf/autoserve_ros2_control.xacro" />
 <xacro:include filename="$(find autoserve_description)/urdf/autoserve.trans" />
 <link name="base_footprint">
   <!-- <collision>
-    <origin xyz="0.0 0.0 0.0055" rpy="0 0 0"/>
-    <geometry>
-      <box size="0.45 0.20 0.01" />
+    <origin xyz="0.0 0.0 0.003" rpy="0 0 0"/>
+    <geometry>
+      <box size="0.4 0.20 0.005" />
     </geometry>
   </collision> -->
@@ -26,14 +25,14 @@
     <material name="plastic_translucent_matte_green"/>
   </visual>
-  <!-- <collision>
+  <collision>
     <origin xyz="0 0 0" rpy="0 0 0"/>
     <geometry>
       <mesh filename="package://autoserve_description/meshes/base_link.stl" scale="0.001 0.001 0.001"/>
     </geometry>
-  </collision> -->
-  <collision>
-    <origin xyz="0.0 0.0 0.006" rpy="0 0 0"/>
-    <geometry>
-      <box size="0.45 0.20 0.01" />
+  </collision>
+  <collision>
+    <origin xyz="0.0 0.0 0.003" rpy="0 0 0"/>
+    <geometry>
+      <box size="0.45 0.20 0.005" />
     </geometry>
   </collision>
@@ -67,19 +66,19 @@
 <link name="ydlidar">
   <inertial>
-    <origin xyz="-2.7755575615628914e-17 -1.7308971658813632e-16 -0.012774955364728169" rpy="0 0 0"/>
-    <mass value="0.09117240534114449"/>
-    <inertia ixx="2.9e-05" iyy="2.9e-05" izz="4.9e-05" ixy="-0.0" iyz="-0.0" ixz="0.0"/>
-  </inertial>
-  <visual>
-    <origin xyz="-0.1632 0.0 -0.267" rpy="0 0 0"/>
-    <geometry>
-      <mesh filename="package://autoserve_description/meshes/ydlidar_v1_1.stl" scale="0.00102 0.00102 0.00102"/>
+    <origin xyz="-0.030294099570319616 0.03099999999999979 0.037701142222791084" rpy="0 0 0"/>
+    <mass value="1.1515616542314233"/>
+    <inertia ixx="0.000489" iyy="0.000861" izz="0.000987" ixy="-0.0" iyz="0.0" ixz="-0.000148"/>
+  </inertial>
+  <visual>
+    <origin xyz="-0.162 0.0 -0.25" rpy="0 0 0"/>
+    <geometry>
+      <mesh filename="package://autoserve_description/meshes/yd_lidar_v1_1.stl" scale="0.001 0.001 0.001"/>
     </geometry>
     <material name="plastic_translucent_matte_blue"/>
   </visual>
   <collision>
-    <origin xyz="-0.1632 0.0 -0.267" rpy="0 0 0"/>
-    <geometry>
-      <mesh filename="package://autoserve_description/meshes/ydlidar_v1_1.stl" scale="0.00102 0.00102 0.00102"/>
+    <origin xyz="-0.162 0.0 -0.25" rpy="0 0 0"/>
+    <geometry>
+      <mesh filename="package://autoserve_description/meshes/yd_lidar_v1_1.stl" scale="0.001 0.001 0.001"/>
     </geometry>
   </collision>
@@ -231,10 +230,10 @@
 </joint>
 <joint name="base2lidar" type="fixed">
-  <origin xyz="0.16 0.0 0.262" rpy="0 0 0"/>
+  <origin xyz="0.162 0.0 0.25" rpy="0 0 0"/>
   <parent link="base_link"/>
   <child link="ydlidar"/>
 </joint>
 <joint name="base2camera_1" type="fixed">
-  <origin xyz="0.2 -0.0 0.1755" rpy="0 0 0"/>
+  <origin xyz="0.2 -0.0 0.1705" rpy="0 0 0"/>
   <parent link="base_link"/>
   <child link="depth_camera_1"/>

Commit message: Added perception image subscriber script

File: autoserve_description/urdf/autoserve.xacro (robot description, xacro)
@@ -239,14 +239,14 @@
   <child link="depth_camera_1"/>
 </joint>
-<joint name="base2camera_2" type="fixed">
+<!-- <joint name="base2camera_2" type="fixed">
   <origin xyz="0.105108 -0.0 0.771167" rpy="0 0 0"/>
-  <parent link="base_link"/>
-  <child link="depth_camera_2"/>
-</joint>
-<!-- <joint name="base2camera_2" type="fixed">
-  <origin xyz="0.105108 -0.0 1.3" rpy="0 0 0"/>
   <parent link="base_link"/>
   <child link="depth_camera_2"/>
 </joint> -->
+<joint name="base2camera_2" type="fixed">
+  <origin xyz="0.105108 -0.0 1.3" rpy="0 0 0"/>
+  <parent link="base_link"/>
+  <child link="depth_camera_2"/>
+</joint>
 <joint name="base2rightw" type="continuous">
   <origin xyz="0.0 -0.1659 0.05" rpy="0 0 0"/>
@@ -262,17 +262,17 @@
 </joint>
 <!-- prismatic -->
-<joint name="base2plate_1" type="fixed">
+<joint name="base2plate_1" type="prismatic">
   <origin xyz="0.0 -0.0 0.303" rpy="0 0 0"/>
   <parent link="base_link"/>
   <child link="plate_1"/>
-  <!-- <axis xyz="1.0 -0.0 -0.0"/>
-  <limit upper="0.08" lower="-0.08" effort="100" velocity="100"/> -->
-</joint>
-<joint name="base2plate_2" type="fixed">
+  <axis xyz="1.0 -0.0 -0.0"/>
+  <limit upper="0.08" lower="-0.08" effort="100" velocity="100"/>
+</joint>
+<joint name="base2plate_2" type="prismatic">
   <origin xyz="0.0 -0.0 0.533" rpy="0 0 0"/>
   <parent link="base_link"/>
   <child link="plate_2"/>
-  <!-- <axis xyz="1.0 -0.0 -0.0"/>
-  <limit upper="0.08" lower="-0.08" effort="100" velocity="100"/> -->
+  <axis xyz="1.0 -0.0 -0.0"/>
+  <limit upper="0.08" lower="-0.08" effort="100" velocity="100"/>
 </joint>
 </robot>

File: autoserve_description/urdf/autoserve_gazebo.xacro (robot description, xacro)
@@ -154,5 +154,5 @@
         <clip>
           <near>0.05</near>
-          <far>10</far>
+          <far>30</far>
         </clip>
       </camera>
@@ -191,5 +191,5 @@
         <clip>
           <near>0.05</near>
-          <far>10</far>
+          <far>30</far>
         </clip>
       </camera>

Commit message: Added 3d mapping and octo2grid and navigation

File: autoserve_description/urdf/autoserve.xacro (robot description, xacro)
@@ -84,5 +84,5 @@
   </collision>
 </link>
-<link name="depth_camera_1">
+<link name="camera_link">
   <inertial>
     <origin xyz="0.011951472788559625 0.022747274204167237 -6.086448440437153e-05" rpy="0 0 0"/>
@@ -104,4 +104,11 @@
   </collision>
 </link>
+<link name="camera_link_optical"/>
+<joint name="camera2camera_1" type="fixed">
+  <parent link="camera_link"/>
+  <child link="camera_link_optical"/>
+  <origin xyz="0 0 0" rpy="-1.5708 0 -1.5708"/>
+  <axis xyz="0 0 0"/>
+</joint>
 <link name="depth_camera_2">
   <inertial>
@@ -237,5 +244,5 @@
   <origin xyz="0.2 -0.0 0.1705" rpy="0 0 0"/>
   <parent link="base_link"/>
-  <child link="depth_camera_1"/>
+  <child link="camera_link"/>
 </joint>
 <!-- <joint name="base2camera_2" type="fixed">

File: autoserve_description/urdf/autoserve_gazebo.xacro (robot description, xacro)
@@ -120,5 +120,5 @@
         </scan>
         <range>
-          <min>0.5</min>
+          <min>0.3</min>
           <max>30.0</max>
           <resolution>0.01</resolution>
@@ -140,10 +140,10 @@
     </sensor>
   </gazebo>
-  <gazebo reference="depth_camera_1">
-    <sensor name="camera_1" type="depth">
+  <gazebo reference="camera_link">
+    <sensor name="camera" type="depth">
       <pose> 0 0 0 0 0 0</pose>
       <visualize>true</visualize>
       <update_rate>60.0</update_rate>
-      <camera name="depth_camera_1">
+      <camera name="camera_link">
         <horizontal_fov>1.047198</horizontal_fov>
         <image>
@@ -154,5 +154,5 @@
         <clip>
           <near>0.05</near>
-          <far>30</far>
+          <far>50</far>
         </clip>
       </camera>
@@ -161,7 +161,7 @@
         <alwaysOn>true</alwaysOn>
         <updateRate>0.0</updateRate>
-        <frame_name>depth_camera_1</frame_name>
+        <frame_name>camera_link_optical</frame_name>
         <pointCloudCutoff>0.1</pointCloudCutoff>
-        <pointCloudCutoffMax>10.0</pointCloudCutoffMax>
+        <pointCloudCutoffMax>50.0</pointCloudCutoffMax>
         <distortionK1>0</distortionK1>
         <distortionK2>0</distortionK2>
