Commit message: Trying gz custom sensors

File: autoserve_description/urdf/autoserve_gazebo.xacro (robot description, xacro)
@@ -1,9 +1,9 @@
 <?xml version="1.0"?>
-<robot name="autoserve" xmlns:xacro="http://ros.org/wiki/xacro">
+<robot name="autoserve" xmlns:xacro="http://ros.org/wiki/xacro" xmlns:gz="http://gazebosim.org/schemas/ignition/1.0">
 <xacro:property name="base_link" value="Gazebo/Red" />
 <xacro:property name="wheels" value="Gazebo/Black" />
-<xacro:property name="imu" value="Gazebo/PurpleGlow" />
+<!-- <xacro:property name="imu" value="Gazebo/PurpleGlow" />
 <xacro:property name="lidar" value="Gazebo/BlueGlow" />
-<xacro:property name="depth_cam" value="Gazebo/TurquoiseGlow" />
+<xacro:property name="depth_cam" value="Gazebo/TurquoiseGlow" /> -->
 <xacro:property name="plate" value="Gazebo/Green" />
   <!-- Wheels -->
@@ -39,20 +39,20 @@
   </gazebo>
   <gazebo reference="depth_camera_1">
-    <material>${depth_cam}</material>
+    <!-- <material>${depth_cam}</material> -->
     <mu1>0.1</mu1>
     <mu2>0.1</mu2>
   </gazebo>
   <gazebo reference="depth_camera_2">
-    <material>${depth_cam}</material>
+    <!-- <material>${depth_cam}</material> -->
     <mu1>0.1</mu1>
     <mu2>0.1</mu2>
   </gazebo>
   <gazebo reference="ydlidar">
-    <material>${lidar}</material>
+    <!-- <material>${lidar}</material> -->
     <mu1>0.1</mu1>
     <mu2>0.1</mu2>
   </gazebo>
   <gazebo reference="imu">
-    <material>${imu}</material>
+    <!-- <material>${imu}</material> -->
     <mu1>0.1</mu1>
     <mu2>0.1</mu2>
@@ -107,39 +107,39 @@
     </sensor>
   </gazebo> -->
-  <!-- <gazebo reference="ydlidar">
-    <sensor type="ray" name="head_hokuyo_sensor">
-      <pose>0 0 0 0 0 0</pose>
-      <visualize>false</visualize>
+  <gazebo reference="base_footprint">
+    <sensor name="an_odometer" type="custom" gz:type="odometer">
+      <always_on>true</always_on>
       <update_rate>30</update_rate>
-      <ray>
-        <scan>
-          <horizontal>
-            <samples>300</samples>
-            <resolution>1</resolution>
-            <min_angle>-3.14</min_angle>
-            <max_angle>3.14</max_angle>
-          </horizontal>
-        </scan>
-        <range>
-          <min>0.3</min>
-          <max>30.0</max>
-          <resolution>0.01</resolution>
-        </range>
-        <noise>
-          <type>gaussian</type>
-          <mean>0.0</mean>
-          <stddev>0.01</stddev>
+      <gz:odometer>
+        <noise type="gaussian">
+          <mean>0.00001</mean>
+          <stddev>0.00001</stddev>
         </noise>
-      </ray>
-      <plugin name="my_ray_sensor_plugin" filename="libgazebo_ros_ray_sensor.so">
-        <ros>
-          <remapping>~/out:=scan</remapping>
-        </ros>
-        <output_type>sensor_msgs/LaserScan</output_type>
-        <min_intensity>100.0</min_intensity>
-        <frame_name>ydlidar</frame_name>
-      </plugin>
-    </sensor>
-  </gazebo> -->
+      </gz:odometer>
+    </sensor>
+  </gazebo>
+  <gazebo reference="ydlidar">
+    <material>Gazebo/Black</material>
+    <sensor name="laser" type="gpu_lidar">
+        <pose> 0 0 0 0 0 0 </pose>
+        <visualize>true</visualize>
+        <update_rate>10</update_rate>
+        <lidar>
+            <scan>
+                <horizontal>
+                    <samples>360</samples>
+                    <min_angle>-3.14</min_angle>
+                    <max_angle>3.14</max_angle>
+                </horizontal>
+            </scan>
+            <range>
+                <min>0.3</min>
+                <max>12</max>
+            </range>
+        </lidar>
+        <topic>scan</topic>
+        <gz_frame_id>ydlidar</gz_frame_id>
+    </sensor>
+  </gazebo>
   <!-- <gazebo reference="camera_link">
     <sensor name="camera" type="depth">
